File: _autosave-van-sao.sch (KiCad schematic (older format))
At the start: 5 parts, among them X1 Badgelife_shitty_connector

Commit message: final for first production run
Parts:
- BT1: footprint (none) -> Battery:Battery_Panasonic_CR2032-VS1N_Vertical_CircularHoles
Connections:
- wire segments 17 -> 15
Changed lines of the file:
@@
 	3850 3000 3850 5150
-Wire Wire Line
-	3850 5150 3300 5150
 Wire Wire Line
 	2850 5150 2850 4850
@@
 F 0 "BT1" H 1568 4046 50  0000 L CNN
 F 1 "Battery_Cell" H 1568 3955 50  0000 L CNN
-F 2 "" V 1450 4010 50  0001 C CNN
+F 2 "Battery:Battery_Panasonic_CR2032-VS1N_Vertical_CircularHoles" V 1450 4010 50  0001 C CNN
 F 3 "~" V 1450 4010 50  0001 C CNN
 	1    1450 3950
@@
 Text Label 2600 4650 0    50   ~ 0
 VDD
-Wire Wire Line
-	3300 5150 3300 5350
-Connection ~ 3300 5150
-Wire Wire Line
-	3300 5150 2850 5150
 Wire Wire Line
 	1450 5150 2850 5150
@@
 Wire Wire Line
 	2400 4250 2400 4650
+Wire Wire Line
+	2850 5150 3850 5150
 $EndSCHEMATC
