File: van-sao.sch (KiCad schematic (older format))
At the start: 4 parts, among them X1 Badgelife_shitty_connector

Commit message: getting svg2shenzen artwork implemented
Parts:
- D1, D2: footprint LED_SMD:LED_1206_3216Metric_ReverseMount_Hole1.8x2.4mm -> LTST-C230TBKT:LED_LTST-C235KGKRKT
Changed lines of the file:
@@
 EESchema Schematic File Version 4
+LIBS:van-sao-cache
 EELAYER 29 0
 EELAYER END
@@
 F 0 "D1" H 2993 2745 50  0000 C CNN
 F 1 "LED" H 2993 2836 50  0000 C CNN
-F 2 "LED_SMD:LED_1206_3216Metric_ReverseMount_Hole1.8x2.4mm" H 3000 3000 50  0001 C CNN
+F 2 "LTST-C230TBKT:LED_LTST-C235KGKRKT" H 3000 3000 50  0001 C CNN
 F 3 "~" H 3000 3000 50  0001 C CNN
 	1    3000 3000
@@
 F 0 "D2" H 3693 2745 50  0000 C CNN
 F 1 "LED" H 3693 2836 50  0000 C CNN
-F 2 "LED_SMD:LED_1206_3216Metric_ReverseMount_Hole1.8x2.4mm" H 3700 3000 50  0001 C CNN
+F 2 "LTST-C230TBKT:LED_LTST-C235KGKRKT" H 3700 3000 50  0001 C CNN
 F 3 "~" H 3700 3000 50  0001 C CNN
 	1    3700 3000

Commit message: final for first production run
Parts:
- added BT1: Battery_Cell, symbol Device:Battery_Cell
- D1, D2: footprint LTST-C230TBKT:LED_LTST-C235KGKRKT -> LED_SMD:LED_1206_3216Metric
- R1: footprint Resistor_SMD:R_1206_3216Metric -> Resistor_SMD:R_0805_2012Metric
Connections:
- net VDD: now reaches R1.2, X1.1 (VDD)
- net VDD: now also BT1.1 (+)
- net at D2.1 (K), X1.2 (GND): now also BT1.2 (-)
Changed lines of the file:
@@
 F 0 "D1" H 2993 2745 50  0000 C CNN
 F 1 "LED" H 2993 2836 50  0000 C CNN
-F 2 "LTST-C230TBKT:LED_LTST-C235KGKRKT" H 3000 3000 50  0001 C CNN
+F 2 "LED_SMD:LED_1206_3216Metric" H 3000 3000 50  0001 C CNN
 F 3 "~" H 3000 3000 50  0001 C CNN
 	1    3000 3000
@@
 F 0 "D2" H 3693 2745 50  0000 C CNN
 F 1 "LED" H 3693 2836 50  0000 C CNN
-F 2 "LTST-C230TBKT:LED_LTST-C235KGKRKT" H 3700 3000 50  0001 C CNN
+F 2 "LED_SMD:LED_1206_3216Metric" H 3700 3000 50  0001 C CNN
 F 3 "~" H 3700 3000 50  0001 C CNN
 	1    3700 3000
@@
 F 0 "R1" H 2470 3846 50  0000 L CNN
 F 1 "1K" H 2470 3755 50  0000 L CNN
-F 2 "Resistor_SMD:R_1206_3216Metric" V 2330 3800 50  0001 C CNN
+F 2 "Resistor_SMD:R_0805_2012Metric" V 2330 3800 50  0001 C CNN
 F 3 "~" H 2400 3800 50  0001 C CNN
 	1    2400 3800
@@
 	3150 3000 3550 3000
 Wire Wire Line
-	2400 3950 2400 4650
+	2400 3950 2400 4250
 Wire Wire Line
 	2400 4650 2850 4650
@@
 	3850 3000 3850 5150
 Wire Wire Line
-	3850 5150 2850 5150
-Wire Wire Line
 	2850 5150 2850 4850
 NoConn ~ 3750 4650
 NoConn ~ 3750 4850
+$Comp
+L Device:Battery_Cell BT1
+U 1 1 5CE07F40
+P 1450 3950
+F 0 "BT1" H 1568 4046 50  0000 L CNN
+F 1 "Battery_Cell" H 1568 3955 50  0000 L CNN
+F 2 "" V 1450 4010 50  0001 C CNN
+F 3 "~" V 1450 4010 50  0001 C CNN
+	1    1450 3950
+	1    0    0    -1
+$EndComp
+Wire Wire Line
+	1450 3750 1450 3000
+Text Label 1800 3000 0    50   ~ 0
+VDD
+Text Label 2600 4650 0    50   ~ 0
+VDD
+Wire Wire Line
+	1450 5150 2850 5150
+Wire Wire Line
+	1450 4050 1450 5150
+Connection ~ 2850 5150
+Wire Wire Line
+	2000 3000 2000 4250
+Wire Wire Line
+	2000 4250 2400 4250
+Wire Wire Line
+	1450 3000 2000 3000
+Connection ~ 2400 4250
+Wire Wire Line
+	2400 4250 2400 4650
+Wire Wire Line
+	2850 5150 3850 5150
 $EndSCHEMATC
